Commit message: gazebo launcher executable

File: leg1_ws/install/leg1_description/share/leg1_description/urdf/leg1.urdf (robot description, URDF)
Before this commit: robot leg1, 6 links, 6 joints
Links:
- removed link driveleg_1
- removed link lowerleg_virtual
- link base_link: geometry collision mesh filename=file:///home/houndsito/vt-cro/robogamescode/leg1_ws/install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 scale=0.001 0.001 0.001; visual mesh filename=file:///home/houndsito/vt-cro/robogamescode/leg1_ws/install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 scale=0.001 0.001 0.001
- link lowerleg_1: geometry collision mesh filename=file:///home/houndsito/vt-cro/robogamescode/leg1_ws/install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 scale=0.001 0.001 0.001; visual mesh filename=file:///home/houndsito/vt-cro/robogamescode/leg1_ws/install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 scale=0.001 0.001 0.001
- link sphere_1: geometry collision mesh filename=file:///home/houndsito/vt-cro/robogamescode/leg1_ws/install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 scale=0.001 0.001 0.001; visual mesh filename=file:///home/houndsito/vt-cro/robogamescode/leg1_ws/install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 scale=0.001 0.001 0.001
- link upperleg_1: geometry collision mesh filename=file:///home/houndsito/vt-cro/robogamescode/leg1_ws/install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 scale=0.001 0.001 0.001; visual mesh filename=file:///home/houndsito/vt-cro/robogamescode/leg1_ws/install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 scale=0.001 0.001 0.001
Joints:
- removed joint Revolute 9
- removed joint Revolute_10
- removed joint Rigid 14
- removed joint mimic_lowerleg
- added joint Revolute 14: type revolute, parent upperleg_1, child lowerleg_1, origin xyz=-0.15 0.0 0.0 rpy=0 0 0, axis 0.0 0.0 1.0, limit lower=-0.506145 upper=0.191986 effort=100 velocity=100
- joint Rigid 13: origin xyz=-0.0025 -0.1255 0.00875 rpy=0 0 0 -> xyz=-0.0025 -0.0755 0.00875 rpy=0 0 0
